File: pcb/Clock PCB/Clock_PCB.kicad_pcb (KiCad board)
At the start: 2 copper layers, 260 x 60 mm, 20 parts, among them J1 PH_2.0_4_Pin, J10 Conn_01x08_Socket, J11 Conn_01x06_Socket, J12 Conn_01x20_Socket, J13 Conn_01x20_Socket, J2 PH_2.0_4_Pin, J3 Conn_01x02_Pin, J4 Conn_01x08_Socket, J5 Conn_01x08_Socket, J6 Conn_01x05_Socket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

Commit message: KiCad PCB changes - PCB now finished, Design Review pending
Parts:
- removed J10, J4, J5, J8: Conn_01x08_Socket, Connector_PinSocket_2.54mm:PinSocket_1x08_P2.54mm_Vertical
- removed J11, J7: Conn_01x06_Socket, Connector_PinSocket_2.54mm:PinSocket_1x06_P2.54mm_Vertical
- removed J12, J13: Conn_01x20_Socket, Connector_PinSocket_2.54mm:PinSocket_1x20_P2.54mm_Vertical
- removed J6, J9: Conn_01x05_Socket, Connector_PinSocket_2.54mm:PinSocket_1x05_P2.54mm_Vertical
- added H1: MountingHole, MountingHole:MountingHole_3.2mm_M3, F.Cu at (6.50, 6.50)
- added H10: MountingHole, MountingHole:MountingHole_3.2mm_M3, F.Cu at (106.5, 52.5)
- added H11: MountingHole, MountingHole:MountingHole_3.2mm_M3, F.Cu at (152.5, 52.5)
- added H12: MountingHole, MountingHole:MountingHole_3.2mm_M3, F.Cu at (152.5, 6.50)
- added H2: MountingHole, MountingHole:MountingHole_3.2mm_M3, F.Cu at (6.50, 52.5)
- added H3: MountingHole, MountingHole:MountingHole_3.2mm_M3, F.Cu at (52.5, 6.50)
- added H4: MountingHole, MountingHole:MountingHole_3.2mm_M3, F.Cu at (52.5, 52.5)
- added H5: MountingHole, MountingHole:MountingHole_3.2mm_M3, F.Cu at (207.5, 6.50)
- added H6: MountingHole, MountingHole:MountingHole_3.2mm_M3, F.Cu at (253.5, 6.50)
- added H7: MountingHole, MountingHole:MountingHole_3.2mm_M3, F.Cu at (253.5, 52.5)
- added H8: MountingHole, MountingHole:MountingHole_3.2mm_M3, F.Cu at (207.5, 52.5)
- added H9: MountingHole, MountingHole:MountingHole_3.2mm_M3, F.Cu at (106.5, 6.50)
- U1: footprint Module:RaspberryPi_Pico_Common_Unspecified -> custom_footprint_library:RaspberryPi_Pico_Common_THT_Header
- moved U1 29.2 mm to (80.0, 5.00)
- moved J3 5.00 mm to (165.0, 53.0)
- moved SW1 5.00 mm to (165.0, 12.0)
- moved J1 3.06 mm to (193.0, 53.3)
- moved U3 2.00 mm to (63.0, 30.0)
- moved J2 0.96 mm to (199.0, 7.00)
Connections:
- J1 pad 1: +5V -> GND
- J1 pad 2: +5V -> /SCL_I2C
- J1 pad 3: +5V -> /SDA_I2C
- J2 pad 2: +5V -> /SDA_I2C
- J2 pad 3: +5V -> /SCL_I2C
- J2 pad 4: +5V -> GND
- J3 pad 2: +5V -> GND
- M1 pad 1: /M1A_1 -> /M1B_3
- M1 pad 2: /M1A_2 -> /M1B_4
- M1 pad 3: /M1A_3 -> /M1A_1
- M1 pad 4: /M1A_4 -> /M1A_2
- M1 pad 5: (no net) -> /M1B_2
- M1 pad 6: (no net) -> /M1B_1
- M1 pad 7: (no net) -> /M1A_4
- M1 pad 8: (no net) -> /M1A_3
- M2 pad 1: /M2A_1 -> /M2B_3
- M2 pad 2: /M2A_2 -> /M2B_4
- M2 pad 3: /M2A_3 -> /M2A_1
- M2 pad 4: /M2A_4 -> /M2A_2
- M2 pad 5: (no net) -> /M2B_2
- M2 pad 6: (no net) -> /M2B_1
- M2 pad 7: (no net) -> /M2A_4
- M2 pad 8: (no net) -> /M2A_3
- M3 pad 1: /M3A_1 -> /M3B_3
- M3 pad 2: /M3A_2 -> /M3B_4
- M3 pad 3: /M3A_3 -> /M3A_1
- M3 pad 4: /M3A_4 -> /M3A_2
- M3 pad 5: (no net) -> /M3B_2
- M3 pad 6: (no net) -> /M3B_1
- M3 pad 7: (no net) -> /M3A_4
- M3 pad 8: (no net) -> /M3A_3
- SW1 pad 1: +5V -> GND
- SW1 pad 2: +5V -> GND
- SW1 pad 3: +5V -> GND
- SW1 pad 4: +5V -> GND
- U1 pad 13: +5V -> GND
- U1 pad 18: +5V -> GND
- U1 pad 23: +5V -> GND
- U1 pad 28: +5V -> GND
- U1 pad 3: +5V -> GND
- U1 pad 33: +5V -> GND
- U1 pad 38: +5V -> GND
- U1 pad 6: +5V -> /SDA_I2C
- U1 pad 7: +5V -> /SCL_I2C
- U1 pad 8: +5V -> GND
- U2 pad 26: +5V -> GND
- U3 pad 26: +5V -> GND
Routing:
- net GND: track 0.00 -> 343.3 mm, vias 0 -> 5
- net +5V: track 0.00 -> 235.8 mm, vias 0 -> 2
- net /SCL_I2C: track 0.00 -> 170.4 mm, vias 0 -> 1
- net /SDA_I2C: track 0.00 -> 168.8 mm, vias 0 -> 1
- net Net-(U1-GPIO21): track 0.00 -> 129.1 mm, vias 0 -> 1
- net Net-(U1-GPIO20): track 0.00 -> 124.2 mm, vias 0 -> 1
- net /M2B_SCX: track 0.00 -> 123.4 mm, vias 0 -> 1
- net /M2B_DIR: track 0.00 -> 120.4 mm
- net RST: track 0.00 -> 113.9 mm, vias 0 -> 2
- net Net-(U1-GPIO18): track 0.00 -> 102.2 mm, vias 0 -> 2
- net Net-(U1-GPIO19): track 0.00 -> 101.5 mm, vias 0 -> 2
- net /M2A_DIR: track 0.00 -> 101.5 mm, vias 0 -> 2
- net /M1B_DIR: track 0.00 -> 101.4 mm, vias 0 -> 1
- net /M2A_SCX: track 0.00 -> 101.2 mm
- net /M1A_SCX: track 0.00 -> 100.4 mm, vias 0 -> 1
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Other:
- outline, holes or cut-outs redrawn
