File: pcb/Clock PCB/Clock_PCB.kicad_sch (KiCad schematic)
At the start: 1 part

Commit message: Clock PCB development
Parts:
- added J1, J2: PH_2.0_4_Pin, Connector_JST:JST_PH_S4B-PH-K_1x04_P2.00mm_Horizontal, symbol Connector:Conn_01x04_Pin
- added J10, J4, J5, J8: Conn_01x08_Socket, Connector_PinSocket_2.54mm:PinSocket_1x08_P2.54mm_Vertical, symbol Connector:Conn_01x08_Socket
- added J11, J7: Conn_01x06_Socket, Connector_PinSocket_2.54mm:PinSocket_1x06_P2.54mm_Vertical, symbol Connector:Conn_01x06_Socket
- added J12, J13: Conn_01x20_Socket, Connector_PinSocket_2.54mm:PinSocket_1x20_P2.54mm_Vertical, symbol Connector:Conn_01x20_Socket
- added J3: Conn_01x02_Pin, TerminalBlock_Phoenix:TerminalBlock_Phoenix_MKDS-1,5-2-5.08_1x02_P5.08mm_Horizontal, symbol Connector:Conn_01x02_Pin
- added J6, J9: Conn_01x05_Socket, Connector_PinSocket_2.54mm:PinSocket_1x05_P2.54mm_Vertical, symbol Connector:Conn_01x05_Socket
- added M1, M2, M3: ~, custom_footprint_library:BKA30D-R5, symbol custom_symbol_library:BKA30D-R5
- added SW1: SW_DIP_x04, Button_Switch_THT:SW_DIP_SPSTx04_Slide_9.78x12.34mm_W7.62mm_P2.54mm, symbol Switch:SW_DIP_x04
- added U2, U3: VID6606, custom_footprint_library:SpeedoDrive, symbol custom_symbol_library:SpeedoDrive
- renumbered A1 to U1
Connections:
- net M1A_SCX: now reaches U1.1 (GPIO0)
- net M1A_SCX: now also J6.4 (Pin_4), J9.4 (Pin_4), U2.20 (SA)
- net M2B_DIR: now reaches U1.10 (GPIO7)
- net M2B_DIR: now also J11.4 (Pin_4), J7.4 (Pin_4), U2.25 (DD)
- net M3A_SCX: now reaches U1.11 (GPIO8)
- net M3A_SCX: now also U3.20 (SA)
- net M3A_DIR: now reaches U1.12 (GPIO9)
- net M3A_DIR: now also U3.19 (DA)
- net +5V: now reaches U1.13 (GND), U1.18 (GND), U1.23 (GND), U1.28 (GND), U1.3 (GND), U1.38 (GND), U1.8 (GND)
- net +5V: now also U1.33 (AGND), U1.40 (VBUS), U1.6 (GPIO4), U1.7 (GPIO5), J1.1 (Pin_1), J1.2 (Pin_2), J1.3 (Pin_3), J1.4 (Pin_4), J11.5 (Pin_5), J11.6 (Pin_6), J2.1 (Pin_1), J2.2 (Pin_2), J2.3 (Pin_3), J2.4 (Pin_4), J3.1 (Pin_1), J3.2 (Pin_2), J7.5 (Pin_5), J7.6 (Pin_6), SW1.1, SW1.2, SW1.3, SW1.4, U2.26 (GND), U2.27 (VCC), U3.26 (GND), U3.27 (VCC)
- net M3B_SCX: now reaches U1.14 (GPIO10)
- net M3B_SCX: now also U3.18 (SB)
- net M3B_DIR: now reaches U1.15 (GPIO11)
- net M3B_DIR: now also U3.17 (DB)
- net M1A_DIR: now reaches U1.2 (GPIO1)
- net M1A_DIR: now also J6.3 (Pin_3), J9.3 (Pin_3), U2.19 (DA)
- net at U1.24 (GPIO18): now also SW1.8
- net at U1.25 (GPIO19): now also SW1.7
- net at U1.26 (GPIO20): now also SW1.6
- net at U1.27 (GPIO21): now also SW1.5
- net RST: now reaches U1.29 (GPIO22)
- net RST: now also J6.5 (Pin_5), J9.5 (Pin_5), U2.21 (RST), U3.21 (RST)
- net M2A_SCX: now reaches U1.31 (GPIO26_ADC0)
- net M2A_SCX: now also J11.1 (Pin_1), J7.1 (Pin_1), U2.22 (SC)
- net M2A_DIR: now reaches U1.32 (GPIO27_ADC1)
- net M2A_DIR: now also J11.2 (Pin_2), J7.2 (Pin_2), U2.23 (DC)
- net M1B_SCX: now reaches U1.4 (GPIO2)
- net M1B_SCX: now also J6.2 (Pin_2), J9.2 (Pin_2), U2.18 (SB)
- net M1B_DIR: now reaches U1.5 (GPIO3)
- net M1B_DIR: now also J6.1 (Pin_1), J9.1 (Pin_1), U2.17 (DB)
- net M2B_SCX: now reaches U1.9 (GPIO6)
- net M2B_SCX: now also J11.3 (Pin_3), J7.3 (Pin_3), U2.24 (SD)
- new net M1A_1: J4.4 (Pin_4), J8.4 (Pin_4), M1.1, U2.4 (A1)
- new net M1A_2: J4.3 (Pin_3), J8.3 (Pin_3), M1.2, U2.3 (A2)
- new net M1A_3: J4.2 (Pin_2), J8.2 (Pin_2), M1.3, U2.2 (A3)
- new net M1A_4: J4.1 (Pin_1), J8.1 (Pin_1), M1.4, U2.1 (A4)
- new net M1B_1: J10.4 (Pin_4), J5.4 (Pin_4), M1.1, U2.12 (B1)
- new net M1B_2: J10.3 (Pin_3), J5.3 (Pin_3), M1.2, U2.11 (B2)
- new net M1B_3: J10.2 (Pin_2), J5.2 (Pin_2), M1.3, U2.10 (B3)
- new net M1B_4: J10.1 (Pin_1), J5.1 (Pin_1), M1.4, U2.9 (B4)
- new net M2A_1: J10.5 (Pin_5), J5.5 (Pin_5), M2.1, U2.13 (C1)
- new net M2A_2: J10.6 (Pin_6), J5.6 (Pin_6), M2.2, U2.14 (C2)
- new net M2A_3: J10.7 (Pin_7), J5.7 (Pin_7), M2.3, U2.15 (C3)
- new net M2A_4: J10.8 (Pin_8), J5.8 (Pin_8), M2.4, U2.16 (C4)
- new net M2B_1: J4.5 (Pin_5), J8.5 (Pin_5), M2.1, U2.5 (D1)
- new net M2B_2: J4.6 (Pin_6), J8.6 (Pin_6), M2.2, U2.6 (D2)
- new net M2B_3: J4.7 (Pin_7), J8.7 (Pin_7), M2.3, U2.7 (D3)
- new net M2B_4: J4.8 (Pin_8), J8.8 (Pin_8), M2.4, U2.8 (D4)
- new net M3A_1: M3.1, U3.4 (A1)
- new net M3A_2: M3.2, U3.3 (A2)
- new net M3A_3: M3.3, U3.2 (A3)
- new net M3A_4: M3.4, U3.1 (A4)
- new net M3B_1: M3.1, U3.12 (B1)
- new net M3B_2: M3.2, U3.11 (B2)
- new net M3B_3: M3.3, U3.10 (B3)
- new net M3B_4: M3.4, U3.9 (B4)
Other:
- moved on the sheet: U1

Commit message: KiCad PCB changes - PCB now finished, Design Review pending
Parts:
- removed J10, J4, J5, J8: Conn_01x08_Socket, Connector_PinSocket_2.54mm:PinSocket_1x08_P2.54mm_Vertical, symbol Connector:Conn_01x08_Socket
- removed J11, J7: Conn_01x06_Socket, Connector_PinSocket_2.54mm:PinSocket_1x06_P2.54mm_Vertical, symbol Connector:Conn_01x06_Socket
- removed J12, J13: Conn_01x20_Socket, Connector_PinSocket_2.54mm:PinSocket_1x20_P2.54mm_Vertical, symbol Connector:Conn_01x20_Socket
- removed J6, J9: Conn_01x05_Socket, Connector_PinSocket_2.54mm:PinSocket_1x05_P2.54mm_Vertical, symbol Connector:Conn_01x05_Socket
- added H1, H10, H11, H12, H2, H3, H4, H5, H6, H7, H8, H9: MountingHole, MountingHole:MountingHole_3.2mm_M3, symbol Mechanical:MountingHole
- U1: footprint Module:RaspberryPi_Pico_Common_Unspecified -> custom_footprint_library:RaspberryPi_Pico_Common_THT_Header
Connections:
- net +5V: no longer J1.1 (Pin_1), J1.2 (Pin_2), J1.3 (Pin_3), J2.2 (Pin_2), J2.3 (Pin_3), J2.4 (Pin_4), J3.2 (Pin_2), SW1.1, SW1.2, SW1.3, SW1.4, U1.13 (GND), U1.18 (GND), U1.23 (GND), U1.28 (GND), U1.3 (GND), U1.33 (AGND), U1.38 (GND), U1.6 (GPIO4), U1.7 (GPIO5), U1.8 (GND), U2.26 (GND), U3.26 (GND)
- net M1A_1: now also M1.3 (A1); no longer M1.1
- net M1A_2: now also M1.4 (A2); no longer M1.2
- net M1A_3: now also M1.8 (A3); no longer M1.3
- net M1A_4: now also M1.7 (A4); no longer M1.4
- net M1B_1: now also M1.6 (B1); no longer M1.1
- net M1B_2: now also M1.5 (B2); no longer M1.2
- net M1B_3: now also M1.1 (B3); no longer M1.3
- net M1B_4: now also M1.2 (B4); no longer M1.4
- net M2A_1: now also M2.3 (A1); no longer M2.1
- net M2A_2: now also M2.4 (A2); no longer M2.2
- net M2A_3: now also M2.8 (A3); no longer M2.3
- net M2A_4: now also M2.7 (A4); no longer M2.4
- net M2B_1: now also M2.6 (B1); no longer M2.1
- net M2B_2: now also M2.5 (B2); no longer M2.2
- net M2B_3: now also M2.1 (B3); no longer M2.3
- net M2B_4: now also M2.2 (B4); no longer M2.4
- net M3A_1: now also M3.3 (A1); no longer M3.1
- net M3A_2: now also M3.4 (A2); no longer M3.2
- net M3A_3: now also M3.8 (A3); no longer M3.3
- net M3A_4: now also M3.7 (A4); no longer M3.4
- net M3B_1: now also M3.6 (B1); no longer M3.1
- net M3B_2: now also M3.5 (B2); no longer M3.2
- net M3B_3: now also M3.1 (B3); no longer M3.3
- net M3B_4: now also M3.2 (B4); no longer M3.4
- new net GND: J1.1 (Pin_1), J2.4 (Pin_4), J3.2 (Pin_2), SW1.1, SW1.2, SW1.3, SW1.4, U1.13 (GND), U1.18 (GND), U1.23 (GND), U1.28 (GND), U1.3 (GND), U1.33 (AGND), U1.38 (GND), U1.8 (GND), U2.26 (GND), U3.26 (GND)
- new net SCL_I2C: J1.2 (Pin_2), J2.3 (Pin_3), U1.7 (GPIO5)
- new net SDA_I2C: J1.3 (Pin_3), J2.2 (Pin_2), U1.6 (GPIO4)
- no-connect marks 0 -> 24
Other:
- moved on the sheet: J1, J2, J3
