File: pcb/Clock PCB/KiCad Design Files/Clock_PCB.kicad_pcb (KiCad board)
At the start: 2 copper layers, 260 x 60 mm, 22 parts, among them J1 PH_2.0_4_Pin, J2 PH_2.0_4_Pin, J3 Conn_01x02_Pin, SW1 SW_DIP_x04, U1 RaspberryPi_Pico, U2 VID6606, U3 VID6606

Commit message: Changes on Clock PCB
Routing:
- net +5V: track 235.8 -> 239.6 mm
- net /SDA_I2C: track 168.8 -> 171.7 mm
- net /SCL_I2C: track 170.4 -> 172.2 mm
- net GND: track 343.3 -> 344.3 mm
Other:
- board text added: "+5V"
- board text added: "GND"
- board text added: "SCL"
- board text added: "SDA"

Commit message: Update Clock PCB
Parts:
- M1, M2, M3: value ~ -> BKA30D-R5
- moved J3 49.0 mm to (175.0, 5.00), turned to 180 degrees
- moved SW1 43.3 mm to (170.0, 55.0), turned to 180 degrees
Connections:
- M1 pad 1: /M1B_3 -> /M1A_3
- M1 pad 2: /M1B_4 -> /M1A_4
- M1 pad 3: /M1A_1 -> /M1B_1
- M1 pad 4: /M1A_2 -> /M1B_2
- M1 pad 5: /M1B_2 -> /M1A_2
- M1 pad 6: /M1B_1 -> /M1A_1
- M1 pad 7: /M1A_4 -> /M1B_4
- M1 pad 8: /M1A_3 -> /M1B_3
- M2 pad 1: /M2B_3 -> /M2A_3
- M2 pad 2: /M2B_4 -> /M2A_4
- M2 pad 3: /M2A_1 -> /M2B_1
- M2 pad 4: /M2A_2 -> /M2B_2
- M2 pad 5: /M2B_2 -> /M2A_2
- M2 pad 6: /M2B_1 -> /M2A_1
- M2 pad 7: /M2A_4 -> /M2B_4
- M2 pad 8: /M2A_3 -> /M2B_3
- M3 pad 1: /M3B_3 -> /M3A_3
- M3 pad 2: /M3B_4 -> /M3A_4
- M3 pad 3: /M3A_1 -> /M3B_1
- M3 pad 4: /M3A_2 -> /M3B_2
- M3 pad 5: /M3B_2 -> /M3A_2
- M3 pad 6: /M3B_1 -> /M3A_1
- M3 pad 7: /M3A_4 -> /M3B_4
- M3 pad 8: /M3A_3 -> /M3B_3
Routing:
- net +5V: track 239.6 -> 343.4 mm
- net Net-(U1-GPIO21): track 129.1 -> 68.5 mm, vias 1 -> 0
- net Net-(U1-GPIO20): track 124.2 -> 68.5 mm, vias 1 -> 0
- net GND: track 344.3 -> 387.0 mm, vias 5 -> 3
- net Net-(U1-GPIO18): track 102.2 -> 68.5 mm, vias 2 -> 0
- net Net-(U1-GPIO19): track 101.5 -> 68.5 mm, vias 2 -> 0
- net /M1B_1: track 37.2 -> 68.9 mm, vias 0 -> 1
- net /M1B_2: track 46.0 -> 75.1 mm
- net /M2B_2: track 87.4 -> 61.1 mm
- net /M1A_3: track 37.4 -> 62.5 mm, vias 1 -> 0
- net /M2B_3: track 60.1 -> 35.6 mm
- net /M1A_2: track 62.9 -> 83.7 mm, vias 0 -> 1
- net /M2A_1: track 59.7 -> 40.1 mm
- net /M2A_2: track 59.5 -> 40.7 mm, vias 1 -> 0
- net /M1B_3: track 60.4 -> 79.2 mm
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