File: pcb/Clock PCB/KiCad Design Files/Clock_PCB.kicad_sch (KiCad schematic)
At the start: 22 parts, among them J1 PH_2.0_4_Pin, J2 PH_2.0_4_Pin, J3 Conn_01x02_Pin, SW1 SW_DIP_x04, U1 RaspberryPi_Pico, U2 VID6606, U3 VID6606

Commit message: Update Clock PCB
Connections:
- net M1A_1: now also M1.6 (A1); no longer M1.3 (A1)
- net M1A_2: now also M1.5 (A2); no longer M1.4 (A2)
- net M1A_3: now also M1.1 (A3); no longer M1.8 (A3)
- net M1A_4: now also M1.2 (A4); no longer M1.7 (A4)
- net M1B_1: now also M1.3 (B1); no longer M1.6 (B1)
- net M1B_2: now also M1.4 (B2); no longer M1.5 (B2)
- net M1B_3: now also M1.8 (B3); no longer M1.1 (B3)
- net M1B_4: now also M1.7 (B4); no longer M1.2 (B4)
- net M2A_1: now also M2.6 (A1); no longer M2.3 (A1)
- net M2A_2: now also M2.5 (A2); no longer M2.4 (A2)
- net M2A_3: now also M2.1 (A3); no longer M2.8 (A3)
- net M2A_4: now also M2.2 (A4); no longer M2.7 (A4)
- net M2B_1: now also M2.3 (B1); no longer M2.6 (B1)
- net M2B_2: now also M2.4 (B2); no longer M2.5 (B2)
- net M2B_3: now also M2.8 (B3); no longer M2.1 (B3)
- net M2B_4: now also M2.7 (B4); no longer M2.2 (B4)
- net M3A_1: now also M3.6 (A1); no longer M3.3 (A1)
- net M3A_2: now also M3.5 (A2); no longer M3.4 (A2)
- net M3A_3: now also M3.1 (A3); no longer M3.8 (A3)
- net M3A_4: now also M3.2 (A4); no longer M3.7 (A4)
- net M3B_1: now also M3.3 (B1); no longer M3.6 (B1)
- net M3B_2: now also M3.4 (B2); no longer M3.5 (B2)
- net M3B_3: now also M3.8 (B3); no longer M3.1 (B3)
- net M3B_4: now also M3.7 (B4); no longer M3.2 (B4)
Other:
- moved on the sheet: M1A, M1B, M2A, M2B, M3A, M3B
Changed lines of the file:
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@@
 	(wire
 		(pts
-			(xy 125.73 109.22) (xy 135.89 109.22)
+			(xy 115.57 109.22) (xy 125.73 109.22)
 		)
 		(stroke
@@
 	(wire
 		(pts
-			(xy 125.73 124.46) (xy 135.89 124.46)
+			(xy 115.57 124.46) (xy 125.73 124.46)
 		)
 		(stroke
@@
 	(wire
 		(pts
-			(xy 163.83 124.46) (xy 153.67 124.46)
+			(xy 153.67 124.46) (xy 143.51 124.46)
 		)
 		(stroke
@@
 	(wire
 		(pts
-			(xy 163.83 114.3) (xy 153.67 114.3)
+			(xy 153.67 114.3) (xy 143.51 114.3)
 		)
 		(stroke
@@
 	(wire
 		(pts
-			(xy 125.73 119.38) (xy 135.89 119.38)
+			(xy 115.57 119.38) (xy 125.73 119.38)
 		)
 		(stroke
@@
 	(wire
 		(pts
-			(xy 163.83 109.22) (xy 153.67 109.22)
+			(xy 153.67 109.22) (xy 143.51 109.22)
 		)
 		(stroke
@@
 	(wire
 		(pts
-			(xy 163.83 119.38) (xy 153.67 119.38)
+			(xy 153.67 119.38) (xy 143.51 119.38)
 		)
 		(stroke
@@
 	(wire
 		(pts
-			(xy 125.73 114.3) (xy 135.89 114.3)
+			(xy 115.57 114.3) (xy 125.73 114.3)
 		)
 		(stroke
@@
 		)
 	)
-	(label "M2A_3"
+	(label "M2B_3"
 		(at 104.14 124.46 180)
 		(effects
@@
 		)
 	)
-	(label "M1A_4"
+	(label "M1B_4"
 		(at 54.61 119.38 180)
 		(effects
@@
 		)
 	)
-	(label "M2B_4"
+	(label "M2A_4"
 		(at 66.04 114.3 0)
 		(effects
@@
 		)
 	)
-	(label "M1A_3"
+	(label "M1B_3"
 		(at 54.61 124.46 180)
 		(effects
@@
 		)
 	)
-	(label "M2B_1"
+	(label "M2A_1"
 		(at 104.14 114.3 180)
 		(effects
@@
 		)
 	)
-	(label "M2A_4"
+	(label "M2B_4"
 		(at 104.14 119.38 180)
 		(effects
@@
 		)
 	)
-	(label "M3B_2"
-		(at 163.83 109.22 180)
+	(label "M3A_2"
+		(at 153.67 109.22 180)
 		(effects
 			(font
@@
 		)
 	)
-	(label "M3A_2"
-		(at 125.73 124.46 0)
+	(label "M3B_2"
+		(at 115.57 124.46 0)
 		(effects
 			(font
@@
 		)
 	)
-	(label "M1B_3"
+	(label "M1A_3"
 		(at 16.51 109.22 0)
 		(effects
@@
 		)
 	)
-	(label "M3B_1"
-		(at 163.83 114.3 180)
+	(label "M3A_1"
+		(at 153.67 114.3 180)
 		(effects
 			(font
@@
 		)
 	)
-	(label "M1B_2"
+	(label "M1A_2"
 		(at 54.61 109.22 180)
 		(effects
@@
 		)
 	)
-	(label "M3B_3"
-		(at 125.73 109.22 0)
+	(label "M3A_3"
+		(at 115.57 109.22 0)
 		(effects
 			(font
@@
 		)
 	)
-	(label "M2B_2"
+	(label "M2A_2"
 		(at 104.14 109.22 180)
 		(effects
@@
 		)
 	)
-	(label "M1A_2"
+	(label "M1B_2"
 		(at 16.51 124.46 0)
 		(effects
@@
 		)
 	)
-	(label "M1B_1"
+	(label "M1A_1"
 		(at 54.61 114.3 180)
 		(effects
@@
 		)
 	)
-	(label "M3A_3"
-		(at 163.83 124.46 180)
+	(label "M3B_3"
+		(at 153.67 124.46 180)
 		(effects
 			(font
@@
 		)
 	)
-	(label "M1A_1"
+	(label "M1B_1"
 		(at 16.51 119.38 0)
 		(effects
@@
 		)
 	)
-	(label "M2B_3"
+	(label "M2A_3"
 		(at 66.04 109.22 0)
 		(effects
@@
 		)
 	)
-	(label "M1B_4"
+	(label "M1A_4"
 		(at 16.51 114.3 0)
 		(effects
@@
 		)
 	)
-	(label "M3A_4"
-		(at 163.83 119.38 180)
+	(label "M3B_4"
+		(at 153.67 119.38 180)
 		(effects
 			(font
@@
 		)
 	)
-	(label "M3A_1"
-		(at 125.73 119.38 0)
+	(label "M3B_1"
+		(at 115.57 119.38 0)
 		(effects
 			(font
@@
 		)
 	)
-	(label "M3B_4"
-		(at 125.73 114.3 0)
+	(label "M3A_4"
+		(at 115.57 114.3 0)
 		(effects
 			(font
@@
 		)
 	)
-	(label "M2A_2"
+	(label "M2B_2"
 		(at 66.04 124.46 0)
 		(effects
@@
 		)
 	)
-	(label "M2A_1"
+	(label "M2B_1"
 		(at 66.04 119.38 0)
 		(effects
@@
 	(symbol
 		(lib_id "custom_symbol_library:BKA30D-R5")
-		(at 144.78 116.84 0)
+		(at 134.62 116.84 0)
 		(unit 1)
 		(exclude_from_sim no)
@@
 		(dnp no)
 		(property "Reference" "M3"
-			(at 144.78 127 0)
+			(at 134.62 105.41 0)
 			(effects
 				(font
@@
 		)
 		(property "Value" "~"
-			(at 144.907 116.84 0)
+			(at 134.747 116.84 0)
 			(effects
 				(font
@@
 		)
 		(property "Footprint" "custom_footprint_library:BKA30D-R5"
-			(at 144.78 116.84 0)
+			(at 134.62 116.84 0)
 			(effects
 				(font
@@
 		)
 		(property "Datasheet" ""
-			(at 144.78 116.84 0)
+			(at 134.62 116.84 0)
 			(effects
 				(font
@@
 		)
 		(property "Description" ""
-			(at 144.78 116.84 0)
+			(at 134.62 116.84 0)
 			(effects
 				(font
@@
 	(symbol
 		(lib_id "custom_symbol_library:BKA30D-R5")
-		(at 144.78 116.84 0)
+		(at 134.62 116.84 0)
 		(unit 2)
 		(exclude_from_sim no)
@@
 		(dnp no)
 		(property "Reference" "M3"
-			(at 144.78 105.918 0)
+			(at 134.62 127.508 0)
 			(effects
 				(font
@@
 		)
 		(property "Value" "~"
-			(at 144.78 106.68 0)
+			(at 134.62 106.68 0)
 			(effects
 				(font
@@
 		)
 		(property "Footprint" "custom_footprint_library:BKA30D-R5"
-			(at 144.78 116.84 0)
+			(at 134.62 116.84 0)
 			(effects
 				(font
@@
 		)
 		(property "Datasheet" ""
-			(at 144.78 116.84 0)
+			(at 134.62 116.84 0)
 			(effects
 				(font
@@
 		)
 		(property "Description" ""
-			(at 144.78 116.84 0)
+			(at 134.62 116.84 0)
 			(effects
 				(font
@@
 		(dnp no)
 		(property "Reference" "M2"
-			(at 85.09 105.918 0)
+			(at 84.836 127.762 0)
 			(effects
 				(font
@@
 		(dnp no)
 		(property "Reference" "M2"
-			(at 85.09 127 0)
+			(at 85.344 106.172 0)
 			(effects
 				(font
@@
 		(dnp no)
 		(property "Reference" "M1"
-			(at 35.56 105.918 0)
+			(at 35.56 127.762 0)
 			(effects
 				(font
@@
 		(dnp no)
 		(property "Reference" "M1"
-			(at 35.56 127 0)
+			(at 35.56 106.172 0)
 			(effects
 				(font
